Commit message: Cameras

File: Assets/URDF/puddles.urdf (robot description, URDF)
Before this commit: robot puddles, 29 links, 28 joints
Links:
- removed link puddles/downward_link
- removed link puddles/downward_optical
- removed link puddles/stereo/left_link
- removed link puddles/stereo/left_optical
- removed link puddles/stereo/right_link
- removed link puddles/stereo/right_optical
Joints:
- removed joint puddles/downward_joint
- removed joint puddles/downward_optical_joint
- removed joint puddles/stereo/left_joint
- removed joint puddles/stereo/left_optical_joint
- removed joint puddles/stereo/right_joint
- removed joint puddles/stereo/right_optical_joint
