Commit message: YAML sim scene file, skybox, window icon, above water works

File: c_simulator/collision_files/robots/talos.urdf (robot description, URDF)
Before this commit: robot talos, 1 links, 0 joints
Links:
- link talos: geometry collision box size=0.2 0.05 0.05; collision box size=0.35 0.83 0.55
