Commit message: add table with colliders and update liltank colliders for accuracy

File: c_simulator/collision_files/robots/liltank.urdf (robot description, URDF)
Before this commit: robot liltank, 2 links, 1 joints
Links:
- removed link liltank_drivetrain
- removed link liltank_tank
- added link liltank_link; collision box size=0.21 0.17 0.1; collision box size=0.4 0.17 0.17
Joints:
- removed joint fixed_joint
